File: pcb/split45left/split45left.kicad_pcb (KiCad board)
At the start: 2 copper layers, 133.4 x 81 mm, 56 parts, among them U1 nice_nano

Commit message: final changes for version 0.1
Other:
- board text added: "JLCJLCJLCJLC"
Changed lines of the file:
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@@
   (general
     (thickness 1.6)
-    (drawings 24)
+    (drawings 25)
     (tracks 295)
     (zones 0)
@@
     (aux_axis_origin 0 0)
     (grid_origin 16.66875 14.2875)
-    (visible_elements FFFFEF7F)
+    (visible_elements FFFFFF7F)
     (pcbplotparams
-      (layerselection 0x010fc_ffffffff)
-      (usegerberextensions false)
-      (usegerberattributes true)
-      (usegerberadvancedattributes true)
-      (creategerberjobfile true)
+      (layerselection 0x010f0_ffffffff)
+      (usegerberextensions true)
+      (usegerberattributes false)
+      (usegerberadvancedattributes false)
+      (creategerberjobfile false)
       (excludeedgelayer true)
       (linewidth 0.100000)
@@
       (plotinvisibletext false)
       (padsonsilk false)
-      (subtractmaskfromsilk false)
+      (subtractmaskfromsilk true)
       (outputformat 1)
       (mirror false)
-      (drillshape 1)
+      (drillshape 0)
       (scaleselection 1)
-      (outputdirectory ""))
+      (outputdirectory "gerbers"))
   )
   (net 0 "")
@@
       (effects (font (size 0.38 0.38) (thickness 0.06)))
     )
-    (pad 1 thru_hole roundrect (at 0 0) (size 1.7 1.7) (drill 0.7) (layers *.Cu *.Mask) (roundrect_rratio 0.147059)
+    (pad 1 thru_hole roundrect (at 0 0) (size 1.7 1.7) (drill 0.7) (layers *.Cu *.Mask) (roundrect_rratio 0.1470588235294118)
       (net 44 "Net-(Reset1-Pad1)"))
     (model ${KISYS3DMOD}/Connector_Wire.3dshapes/SolderWire-0.15sqmm_1x01_D0.5mm_OD1.5mm.wrl
@@
       (effects (font (size 0.38 0.38) (thickness 0.06)))
     )
-    (pad 1 thru_hole roundrect (at 0 0) (size 1.7 1.7) (drill 0.7) (layers *.Cu *.Mask) (roundrect_rratio 0.147059)
+    (pad 1 thru_hole roundrect (at 0 0) (size 1.7 1.7) (drill 0.7) (layers *.Cu *.Mask) (roundrect_rratio 0.1470588235294118)
       (net 43 GND))
     (model ${KISYS3DMOD}/Connector_Wire.3dshapes/SolderWire-0.15sqmm_1x01_D0.5mm_OD1.5mm.wrl
@@
     )
   )
+  (gr_text JLCJLCJLCJLC (at 116.68125 91.28125) (layer B.SilkS)
+    (effects (font (size 1 1) (thickness 0.15)) (justify mirror))
+  )
   (gr_text "with love from Old Badger" (at 38.89375 92.86875) (layer B.Mask)
