File: pcb/split45leftbase/split45leftbase.kicad_pcb (KiCad board)
At the start: 2 copper layers, 133.4 x 81 mm, 8 parts

Commit message: final changes for version 0.1
Parts:
- added G***: LOGO, split45:split45, B.Cu at (104.0, 45.2)
- added G***: LOGO, split45:logo, B.Cu at (50.8, 54.8)
Other:
- board text added: "JLCJLCJLCJLC"
