File: pcb/split45rightbase/split45rightbase.kicad_pcb (KiCad board)
At the start: 2 copper layers, 138.1 x 81 mm, 8 parts

Commit message: final changes for version 0.1
Parts:
- added G***: LOGO, split45:split45, B.Cu at (65.9, 45.2)
- added G***: LOGO, split45:logo, B.Cu at (119.1, 54.8)
- added G***: LOGO, split45:withlove, B.Cu at (54.8, 80.2)
Other:
- board text added: "JLCJLCJLCJLC"
